File: electrical/bracelet_rev1/bracelet_rev1.kicad_sch (KiCad schematic)
At the start: 0 parts

Commit message: Many schematic updates
Other:
- note added: "Add a current sense"
- note added: "Button"
- note added: "Haptic Driver"
- note removed: "Battery Connector"
- note removed: "Buzzer"
- note removed: "EN"
- note removed: "Toggle Switch (DIP Switch)"
Changed lines of the file:
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@@
 	)
 	(rectangle
-		(start 120.65 34.29)
-		(end 140.97 54.61)
+		(start 120.65 62.23)
+		(end 140.97 82.55)
 		(stroke
 			(width 0)
@@
 	)
 	(rectangle
-		(start 120.65 62.23)
-		(end 140.97 82.55)
+		(start 207.01 115.316)
+		(end 222.25 130.556)
 		(stroke
 			(width 0)
@@
 	)
 	(rectangle
-		(start 153.67 77.47)
-		(end 166.37 90.17)
+		(start 173.99 59.69)
+		(end 194.31 80.01)
 		(stroke
 			(width 0)
@@
 	)
 	(rectangle
-		(start 173.99 59.69)
-		(end 194.31 80.01)
+		(start 256.54 72.39)
+		(end 271.78 87.63)
 		(stroke
 			(width 0)
@@
 	)
 	(rectangle
-		(start 256.54 72.39)
-		(end 271.78 87.63)
+		(start 256.54 34.29)
+		(end 271.78 49.53)
 		(stroke
 			(width 0)
@@
 	)
 	(rectangle
-		(start 256.54 34.29)
-		(end 271.78 49.53)
+		(start 241.3 115.316)
+		(end 256.54 130.556)
+		(stroke
+			(width 0)
+			(type solid)
+		)
+		(fill
+			(type color)
+			(color 215 255 181 1)
+		)
+	)
+	(rectangle
+		(start 256.54 53.34)
+		(end 271.78 68.58)
 		(stroke
 			(width 0)
@@
 	)
 	(rectangle
-		(start 256.54 110.49)
-		(end 271.78 125.73)
-		(stroke
-			(width 0)
-			(type solid)
-		)
-		(fill
-			(type color)
-			(color 215 255 181 1)
-		)
-	)
-	(rectangle
-		(start 256.54 53.34)
-		(end 271.78 68.58)
-		(stroke
-			(width 0)
-			(type solid)
-		)
-		(fill
-			(type color)
-			(color 255 255 194 1)
-		)
-	)
-	(rectangle
 		(start 109.22 24.13)
 		(end 279.4 132.08)
@@
 		)
 	)
-	(text "Buzzer"
+	(text "Haptic\nDriver"
 		(exclude_from_sim no)
 		(at 264.414 80.518 0)
@@
 		)
 	)
-	(text "Battery\nConnector"
-		(exclude_from_sim no)
-		(at 160.528 84.074 0)
-		(effects
-			(font
-				(size 1.27 1.27)
-			)
-		)
-	)
 	(text "RGB LED\n(WS2812)"
 		(exclude_from_sim no)
@@
 		)
 	)
-	(text "EN"
-		(exclude_from_sim no)
-		(at 148.082 39.624 0)
+	(text "I2C"
+		(exclude_from_sim no)
+		(at 248.666 59.944 0)
 		(effects
 			(font
@@
 	(text "RF Antenna\n(Layout\nComponent)"
 		(exclude_from_sim no)
-		(at 264.16 118.364 0)
+		(at 248.92 123.19 0)
 		(effects
 			(font
@@
 		)
 	)
+	(text "Button"
+		(exclude_from_sim no)
+		(at 214.63 123.19 0)
+		(effects
+			(font
+				(size 1.27 1.27)
+			)
+		)
+	)
 	(text "Battery\n(External\nComponent)"
 		(exclude_from_sim no)
@@
 		)
 	)
-	(text "Toggle Switch\n(DIP Switch)"
-		(exclude_from_sim no)
-		(at 130.81 44.704 0)
-		(effects
-			(font
-				(size 1.27 1.27)
-			)
-		)
-	)
 	(text "Battery Charger IC"
 		(exclude_from_sim no)
@@
 		)
 	)
+	(text "Add a current sense"
+		(exclude_from_sim no)
+		(at 210.566 73.914 90)
+		(effects
+			(font
+				(size 1.27 1.27)
+			)
+		)
+	)
 	(text "Heart Rate\nSensor"
 		(exclude_from_sim no)
@@
 	(polyline
 		(pts
+			(xy 142.24 77.47) (xy 140.97 78.74)
+		)
+		(stroke
+			(width 0)
+			(type default)
+		)
+	)
+	(polyline
+		(pts
 			(xy 241.3 62.23) (xy 240.03 60.96)
 		)
@@
 	(polyline
 		(pts
-			(xy 172.72 80.01) (xy 173.99 78.74)
+			(xy 177.8 38.1) (xy 176.53 39.37)
 		)
 		(stroke
@@
 	(polyline
 		(pts
+			(xy 142.24 80.01) (xy 140.97 78.74)
+		)
+		(stroke
+			(width 0)
+			(type default)
+		)
+	)
+	(polyline
+		(pts
 			(xy 148.59 50.8) (xy 156.21 50.8)
 		)
@@
 	(polyline
 		(pts
+			(xy 228.6 100.33) (xy 227.33 99.06)
+		)
+		(stroke
+			(width 0)
+			(type default)
+		)
+	)
+	(polyline
+		(pts
 			(xy 241.3 43.18) (xy 240.03 41.91)
 		)
@@
 	(polyline
 		(pts
+			(xy 227.33 99.06) (xy 227.33 123.19)
+		)
+		(stroke
+			(width 0)
+			(type default)
+		)
+	)
+	(polyline
+		(pts
+			(xy 236.22 99.06) (xy 236.22 123.19)
+		)
+		(stroke
+			(width 0)
+			(type default)
+		)
+	)
+	(polyline
+		(pts
+			(xy 177.8 40.64) (xy 176.53 39.37)
+		)
+		(stroke
+			(width 0)
+			(type default)
+		)
+	)
+	(polyline
+		(pts
+			(xy 176.53 39.37) (xy 181.61 39.37)
+		)
+		(stroke
+			(width 0)
+			(type default)
+		)
+	)
+	(polyline
+		(pts
 			(xy 148.59 95.25) (xy 219.71 95.25)
 		)
@@
 	(polyline
 		(pts
+			(xy 236.22 123.19) (xy 241.3 123.19)
+		)
+		(stroke
+			(width 0)
+			(type default)
+		)
+	)
+	(polyline
+		(pts
 			(xy 184.15 59.69) (xy 184.15 44.45)
 		)
@@
 	(polyline
 		(pts
+			(xy 226.06 100.33) (xy 227.33 99.06)
+		)
+		(stroke
+			(width 0)
+			(type default)
+		)
+	)
+	(polyline
+		(pts
 			(xy 187.96 45.72) (xy 189.23 44.45)
 		)
@@
 	(polyline
 		(pts
-			(xy 166.37 78.74) (xy 173.99 78.74)
-		)
-		(stroke
-			(width 0)
-			(type default)
-		)
-	)
-	(polyline
-		(pts
 			(xy 240.03 60.96) (xy 256.54 60.96)
 		)
@@
 	(polyline
 		(pts
-			(xy 140.97 40.64) (xy 156.21 40.64)
-		)
-		(stroke
-			(width 0)
-			(type default)
-		)
-	)
-	(polyline
-		(pts
 			(xy 255.27 40.64) (xy 256.54 41.91)
 		)
@@
 	(polyline
 		(pts
+			(xy 222.25 123.19) (xy 227.33 123.19)
+		)
+		(stroke
+			(width 0)
+			(type default)
+		)
+	)
+	(polyline
+		(pts
 			(xy 148.59 67.31) (xy 173.99 67.31)
 		)
@@
 	(polyline
 		(pts
-			(xy 255.2339 100.6049) (xy 256.5039 99.3349)
+			(xy 255.27 100.33) (xy 256.54 99.06)
 		)
 		(stroke
@@
 	(polyline
 		(pts
-			(xy 255.2339 98.0649) (xy 256.5039 99.3349)
+			(xy 180.34 39.37) (xy 181.61 39.37)
+		)
+		(stroke
+			(width 0)
+			(type default)
+		)
+	)
+	(polyline
+		(pts
+			(xy 181.61 39.37) (xy 189.23 39.37)
+		)
+		(stroke
+			(width 0)
+			(type default)
+		)
+	)
+	(polyline
+		(pts
+			(xy 255.27 97.79) (xy 256.54 99.06)
 		)
 		(stroke
@@
 	(polyline
 		(pts
-			(xy 154.94 41.91) (xy 156.21 40.64)
-		)
-		(stroke
-			(width 0)
-			(type default)
-		)
-	)
-	(polyline
-		(pts
 			(xy 240.03 92.71) (xy 251.46 92.71)
 		)
@@
 	(polyline
 		(pts
-			(xy 229.87 99.06) (xy 229.87 118.11)
-		)
-		(stroke
-			(width 0)
-			(type default)
-		)
-	)
-	(polyline
-		(pts
-			(xy 229.87 118.11) (xy 256.54 118.11)
-		)
-		(stroke
-			(width 0)
-			(type default)
-		)
-	)
-	(polyline
-		(pts
 			(xy 255.27 81.28) (xy 256.54 80.01)
 		)
@@
 		)
 		(stroke
-			(width 0)
-			(type default)
-		)
-	)
-	(polyline
-		(pts
-			(xy 154.94 39.37) (xy 156.21 40.64)
-		)
-		(stroke
-			(width 0)
-			(type default)
-		)
-	)
-	(polyline
-		(pts
-			(xy 172.72 77.47) (xy 173.99 78.74)
-		)
-		(stroke

Commit message: Mostly finihsed hopefully but still needs clean up anyway
Other:
- note added: "1V8 Regulator (Buck)"
- note added: "Current Sense"
- note removed: "Add a current sense"

Commit message: May updates
Other:
- added sheet Wi-Fi (untitled.kicad_sch)
- note added: "Block Diagram (Rev 1.0)"
- note removed: "Block Diagram"
Changed lines of the file:
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@@
 		)
 	)
-	(text "Block Diagram"
-		(exclude_from_sim no)
-		(at 122.682 21.59 0)
+	(text "Block Diagram (Rev 1.0)"
+		(exclude_from_sim no)
+		(at 109.22 22.86 0)
 		(effects
 			(font
 				(size 2.54 2.54)
 			)
+			(justify left bottom)
 		)
 	)
@@
 				)
 			)
+		)
+	)
+	(sheet
+		(at 19.05 173.482)
+		(size 23.368 14.478)
+		(exclude_from_sim no)
+		(in_bom yes)
+		(on_board yes)
+		(dnp no)
+		(fields_autoplaced yes)
+		(stroke
+			(width 0.1524)
+			(type solid)
+		)
+		(fill
+			(color 0 0 0 0.0000)
+		)
+		(property "Sheetname" "Wi-Fi"
+			(at 19.05 172.7704 0)
+			(effects
+				(font
+					(size 1.27 1.27)
+				)
+				(justify left bottom)
+			)
+		)
+		(property "Sheetfile" "untitled.kicad_sch"
+			(at 19.05 188.5446 0)
+			(effects
+				(font
+					(size 1.27 1.27)
+				)
+				(justify left top)
+			)
+		)
+		(instances
+			(project "bracelet_rev1"
+				(path "/2a7dd2e8-59c9-4d04-9427-958ca4ea7daa"
+					(page "5")
+				)
+			)
