File: electrical/esp_module_rev1/esp_module_rev1/esp_module_rev1.kicad_pcb (KiCad board)
At the start: 2 copper layers, 0 parts

Commit message: Layout attempt
Parts:
- added C1: 10uF, Capacitor_SMD:C_0603_1608Metric_Pad1.08x0.95mm_HandSolder, F.Cu at (144.5, 92.2)
- added C10: 100nF, Capacitor_SMD:C_0603_1608Metric_Pad1.08x0.95mm_HandSolder, F.Cu at (120.8, 84.0)
- added C11: 0u1F, Capacitor_SMD:C_0603_1608Metric_Pad1.08x0.95mm_HandSolder, F.Cu at (118.2, 86.2)
- added C12: 0u1F, Capacitor_SMD:C_0603_1608Metric_Pad1.08x0.95mm_HandSolder, F.Cu at (126.2, 87.9)
- added C13: 1uF, Capacitor_SMD:C_0603_1608Metric_Pad1.08x0.95mm_HandSolder, F.Cu at (128.0, 87.9)
- added C14: 10uF, Capacitor_SMD:C_0603_1608Metric_Pad1.08x0.95mm_HandSolder, F.Cu at (135.2, 89.9)
- added C15: 0u1F, Capacitor_SMD:C_0603_1608Metric_Pad1.08x0.95mm_HandSolder, F.Cu at (132.6, 90.9)
- added C16: 0u1F, Capacitor_SMD:C_0603_1608Metric_Pad1.08x0.95mm_HandSolder, B.Cu at (136.0, 87.5)
- added C17: 0u1F, Capacitor_SMD:C_0603_1608Metric_Pad1.08x0.95mm_HandSolder, B.Cu at (136.0, 90.0)
- added C18: 0u1F, Capacitor_SMD:C_0603_1608Metric_Pad1.08x0.95mm_HandSolder, B.Cu at (136.0, 92.5)
- added C19: 1uF, Capacitor_SMD:C_0603_1608Metric_Pad1.08x0.95mm_HandSolder, B.Cu at (136.0, 95.0)
- added C2: 10uF, Capacitor_SMD:C_0603_1608Metric_Pad1.08x0.95mm_HandSolder, F.Cu at (140.9, 92.5)
- added C20: 100nF, Capacitor_SMD:C_0603_1608Metric_Pad1.08x0.95mm_HandSolder, F.Cu at (120.2, 96.5)
- added C21: 100nF, Capacitor_SMD:C_0603_1608Metric_Pad1.08x0.95mm_HandSolder, F.Cu at (120.2, 98.2)
- added C3: 470nF, Capacitor_SMD:C_0603_1608Metric_Pad1.08x0.95mm_HandSolder, F.Cu at (136.8, 97.8)
- added C4: 470nF, Capacitor_SMD:C_0603_1608Metric_Pad1.08x0.95mm_HandSolder, F.Cu at (136.8, 95.8)
- added C5: 10uF, Capacitor_SMD:C_0603_1608Metric_Pad1.08x0.95mm_HandSolder, F.Cu at (145.5, 77.6)
- added C6: 10uF, Capacitor_SMD:C_0603_1608Metric_Pad1.08x0.95mm_HandSolder, F.Cu at (145.4, 85.9)
- added C7: 10uF, Capacitor_SMD:C_0603_1608Metric_Pad1.08x0.95mm_HandSolder, F.Cu at (119.8, 75.0)
- added C8: 0u1F, Capacitor_SMD:C_0603_1608Metric_Pad1.08x0.95mm_HandSolder, F.Cu at (119.8, 73.0)
- added C9: 100nF, Capacitor_SMD:C_0603_1608Metric_Pad1.08x0.95mm_HandSolder, F.Cu at (117.6, 78.7)
- added D1: LED, LED_SMD:LED_0805_2012Metric_Pad1.15x1.40mm_HandSolder, F.Cu at (144.8, 94.2)
- added D2: 1N5819WS, Diode_SMD:D_SOD-323, F.Cu at (142.7, 75.2)
- added D3: 1N5819WS, Diode_SMD:D_SOD-323, F.Cu at (142.7, 83.2)
- added D4: LED, LED_SMD:LED_1206_3216Metric_Pad1.42x1.75mm_HandSolder, F.Cu at (139.8, 89.0)
- added H1: MountingHole, MountingHole:MountingHole_2.2mm_M2, F.Cu at (112.6, 75.0)
- added H2: MountingHole, MountingHole:MountingHole_2.2mm_M2, F.Cu at (112.6, 93.0)
- added H3: MountingHole, MountingHole:MountingHole_2.2mm_M2, F.Cu at (151.1, 86.8)
- added J1: USB_C_Receptacle_USB2.0_14P, Connector_USB:USB_C_Receptacle_GCT_USB4105-xx-A_16P_TopMnt_Horizontal, F.Cu at (129.1, 103.5)
- added J3: Conn_01x02, Connector_JST:JST_PH_B2B-PH-K_1x02_P2.00mm_Vertical, F.Cu at (149.8, 102.2)
- added Q1: FDN340P, Package_TO_SOT_SMD:SOT-23, F.Cu at (145.7, 75.0)
- added Q2: FDN340P, Package_TO_SOT_SMD:SOT-23, F.Cu at (145.8, 83.2)
- added R1: 0R, Resistor_SMD:R_0603_1608Metric_Pad0.98x0.95mm_HandSolder, F.Cu at (134.2, 96.8)
- added R10: 0R, Resistor_SMD:R_0603_1608Metric_Pad0.98x0.95mm_HandSolder, F.Cu at (114.6, 81.1)
- added R11: 5k1, Resistor_SMD:R_0603_1608Metric_Pad0.98x0.95mm_HandSolder, F.Cu at (118.0, 83.2)
- added R12: 0R, Resistor_SMD:R_0603_1608Metric_Pad0.98x0.95mm_HandSolder, F.Cu at (112.8, 81.1)
- added R13: 5k1, Resistor_SMD:R_0603_1608Metric_Pad0.98x0.95mm_HandSolder, F.Cu at (139.7, 86.8)
- added R14: 5k1, Resistor_SMD:R_0603_1608Metric_Pad0.98x0.95mm_HandSolder, F.Cu at (125.8, 93.2)
- added R15: 5k1, Resistor_SMD:R_0603_1608Metric_Pad0.98x0.95mm_HandSolder, F.Cu at (116.5, 88.4)
- added R16: 5k1, Resistor_SMD:R_0603_1608Metric_Pad0.98x0.95mm_HandSolder, F.Cu at (117.5, 91.2)
- added R17: 5k1, Resistor_SMD:R_0603_1608Metric_Pad0.98x0.95mm_HandSolder, F.Cu at (122.2, 91.8)
- added R18: 200k, Resistor_SMD:R_0603_1608Metric_Pad0.98x0.95mm_HandSolder, F.Cu at (150.2, 92.8)
- added R19: 100k, Resistor_SMD:R_0603_1608Metric_Pad0.98x0.95mm_HandSolder, F.Cu at (150.2, 91.0)
- added R2: 5k1, Resistor_SMD:R_0603_1608Metric_Pad0.98x0.95mm_HandSolder, F.Cu at (141.0, 91.0)
- added R20: 100m, Resistor_SMD:R_0603_1608Metric_Pad0.98x0.95mm_HandSolder, F.Cu at (150.2, 98.5)
- added R21: 0R, Resistor_SMD:R_0603_1608Metric_Pad0.98x0.95mm_HandSolder, F.Cu at (129.8, 88.5)
- added R22: 0R, Resistor_SMD:R_0603_1608Metric_Pad0.98x0.95mm_HandSolder, F.Cu at (117.0, 94.6)
- added R3: 10k, Resistor_SMD:R_0603_1608Metric_Pad0.98x0.95mm_HandSolder, F.Cu at (141.6, 98.0)
- added R4: 5k1, Resistor_SMD:R_0603_1608Metric_Pad0.98x0.95mm_HandSolder, F.Cu at (146.0, 97.2)
- added R5: 5k1, Resistor_SMD:R_0603_1608Metric_Pad0.98x0.95mm_HandSolder, F.Cu at (125.4, 96.9)
- added R6: 0, Resistor_SMD:R_0603_1608Metric_Pad0.98x0.95mm_HandSolder, F.Cu at (150.9, 77.6)
- added R7: 0, Resistor_SMD:R_0603_1608Metric_Pad0.98x0.95mm_HandSolder, F.Cu at (151.1, 83.3)
- added R8: 10k, Resistor_SMD:R_0603_1608Metric_Pad0.98x0.95mm_HandSolder, F.Cu at (145.6, 79.5)
- added R9: 5k1, Resistor_SMD:R_0603_1608Metric_Pad0.98x0.95mm_HandSolder, F.Cu at (120.5, 77.7)
- added SW1: SW_Push, Button_Switch_THT:SW_PUSH_6mm, F.Cu at (143.1, 105.2)
- added SW2: SW_Push, Button_Switch_THT:SW_PUSH_6mm, F.Cu at (121.3, 105.2)
- added U1: MCP73831-2-OT, Package_TO_SOT_SMD:SOT-23-5, F.Cu at (140.8, 95.0)
- added U10: BMP390L, BMP390L:10LGA_2X2X0p75_BOS, F.Cu at (117.0, 97.2)
- added U2: USBLC6-2SC6, Package_TO_SOT_SMD:SOT-23-6, F.Cu at (130.8, 96.4)
- added U3: TLV75533PDBV, Package_TO_SOT_SMD:SOT-23-5, F.Cu at (150.5, 74.9)
- added U4: TLV75518PDBV, Package_TO_SOT_SMD:SOT-23-5, F.Cu at (150.6, 80.6)
- added U5: ESP32-C3-WROOM-02, RF_Module:ESP32-C3-WROOM-02, F.Cu at (131.5, 78.6)
- added U6: TXS0102DCT, Package_SO:SSOP-8_2.95x2.8mm_P0.65mm, F.Cu at (121.2, 89.0)
- added U7: INA180A1, Package_TO_SOT_SMD:SOT-23-5, F.Cu at (150.6, 95.5)
- added U8: LSM6DS3, Package_LGA:LGA-14_3x2.5mm_P0.5mm_LayoutBorder3x4y, F.Cu at (132.6, 88.5)
- added U9: MAX30102, OptoDevice:Maxim_OLGA-14_3.3x5.6mm_P0.8mm, B.Cu at (131.8, 90.2)
Routing:
- net GND: track 0.00 -> 151.6 mm, vias 0 -> 8
- net +BATT: track 0.00 -> 47.7 mm, vias 0 -> 6
- net +3V3: track 0.00 -> 39.6 mm, vias 0 -> 8
- net /BMP_INT: track 0.00 -> 36.2 mm, vias 0 -> 2
- net Net-(D3-K): track 0.00 -> 34.6 mm, vias 0 -> 2
- net /USB_CC2: track 0.00 -> 31.6 mm, vias 0 -> 2
- net /BOOT_SEL_GPIO9: track 0.00 -> 31.5 mm, vias 0 -> 1
- net /VBATT_SENSE: track 0.00 -> 31.2 mm, vias 0 -> 2
- net /CURR_SENSE: track 0.00 -> 30.5 mm, vias 0 -> 2
- net +USB_VBUSF: track 0.00 -> 29.5 mm, vias 0 -> 2
- net +USB_VBUS: track 0.00 -> 27.5 mm
- net /LSM_INT2: track 0.00 -> 27.2 mm, vias 0 -> 2
- net Net-(D2-K): track 0.00 -> 24.9 mm, vias 0 -> 2
- net +1V8: track 0.00 -> 19.0 mm, vias 0 -> 4
- net /LSM_INT1: track 0.00 -> 18.5 mm
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- added copper zone on In2.Cu, net +1V8
- added copper zone on In2.Cu, net +3V3
- added copper zone on In1.Cu, net GND
Other:
- board outline added: 47.2 x 47 mm
- copper layers 2 -> 4
