File: electrical/esp_module_rev1/esp_module_rev1/esp_module_rev1.kicad_sch (KiCad schematic)
At the start: 64 parts, among them J1 USB_C_Receptacle_USB2.0_14P, J2 Conn_01x02, J3 Conn_01x02_Pin, Q1 FDN340P, Q2 FDN340P, SW1 SW_Push, SW2 SW_Push, U1 ESP32-C3-WROOM-02, U10 TXS0102DCT, U2 MCP73831-2-OT, U3 INA180A1, U4 TLV75533PDBV, U5 TLV75518PDBV, U6 MAX30102, U7 LSM6DS3, U8 BMP390L, U9 USBLC6-2SC6

Commit message: Layout attempt
Parts:
- removed J3: Conn_01x02_Pin, symbol Connector:Conn_01x02_Pin
- added H1, H2, H3: MountingHole, MountingHole:MountingHole_2.2mm_M2, symbol Mechanical:MountingHole
- C1, C2, C3, C4, C5, C6, C7, C8: footprint (none) -> Capacitor_SMD:C_0603_1608Metric_Pad1.08x0.95mm_HandSolder
- C10: renamed from C21; footprint (none) -> Capacitor_SMD:C_0603_1608Metric_Pad1.08x0.95mm_HandSolder
- C11: renamed from C12; footprint (none) -> Capacitor_SMD:C_0603_1608Metric_Pad1.08x0.95mm_HandSolder
- C12: renamed from C13; footprint (none) -> Capacitor_SMD:C_0603_1608Metric_Pad1.08x0.95mm_HandSolder
- C13: renamed from C14; footprint (none) -> Capacitor_SMD:C_0603_1608Metric_Pad1.08x0.95mm_HandSolder
- C14: renamed from C10; footprint (none) -> Capacitor_SMD:C_0603_1608Metric_Pad1.08x0.95mm_HandSolder
- C15: renamed from C11; footprint (none) -> Capacitor_SMD:C_0603_1608Metric_Pad1.08x0.95mm_HandSolder
- C16: renamed from C15; footprint (none) -> Capacitor_SMD:C_0603_1608Metric_Pad1.08x0.95mm_HandSolder
- C17: renamed from C16; footprint (none) -> Capacitor_SMD:C_0603_1608Metric_Pad1.08x0.95mm_HandSolder
- C18: renamed from C17; footprint (none) -> Capacitor_SMD:C_0603_1608Metric_Pad1.08x0.95mm_HandSolder
- C19: renamed from C18; footprint (none) -> Capacitor_SMD:C_0603_1608Metric_Pad1.08x0.95mm_HandSolder
- C20: renamed from C19; footprint (none) -> Capacitor_SMD:C_0603_1608Metric_Pad1.08x0.95mm_HandSolder
- C21: renamed from C20; footprint (none) -> Capacitor_SMD:C_0603_1608Metric_Pad1.08x0.95mm_HandSolder
- C9: renamed from C22; footprint (none) -> Capacitor_SMD:C_0603_1608Metric_Pad1.08x0.95mm_HandSolder
- D1: footprint (none) -> LED_SMD:LED_0805_2012Metric_Pad1.15x1.40mm_HandSolder
- D4: footprint (none) -> LED_SMD:LED_1206_3216Metric_Pad1.42x1.75mm_HandSolder
- J3: renamed from J2; footprint (none) -> Connector_JST:JST_PH_B2B-PH-K_1x02_P2.00mm_Vertical
- R1: renamed from R10; footprint (none) -> Resistor_SMD:R_0603_1608Metric_Pad0.98x0.95mm_HandSolder
- R10: renamed from R23; footprint (none) -> Resistor_SMD:R_0603_1608Metric_Pad0.98x0.95mm_HandSolder
- R11: renamed from R17; footprint (none) -> Resistor_SMD:R_0603_1608Metric_Pad0.98x0.95mm_HandSolder
- R12: renamed from R22; footprint (none) -> Resistor_SMD:R_0603_1608Metric_Pad0.98x0.95mm_HandSolder
- R13: renamed from R19; footprint (none) -> Resistor_SMD:R_0603_1608Metric_Pad0.98x0.95mm_HandSolder
- R14: footprint (none) -> Resistor_SMD:R_0603_1608Metric_Pad0.98x0.95mm_HandSolder
- R15: renamed from R13; footprint (none) -> Resistor_SMD:R_0603_1608Metric_Pad0.98x0.95mm_HandSolder
- R16: renamed from R20; footprint (none) -> Resistor_SMD:R_0603_1608Metric_Pad0.98x0.95mm_HandSolder
- R17: renamed from R21; footprint (none) -> Resistor_SMD:R_0603_1608Metric_Pad0.98x0.95mm_HandSolder
- R18: renamed from R8; footprint (none) -> Resistor_SMD:R_0603_1608Metric_Pad0.98x0.95mm_HandSolder
- R19: renamed from R9; footprint (none) -> Resistor_SMD:R_0603_1608Metric_Pad0.98x0.95mm_HandSolder
- R2: renamed from R3; footprint (none) -> Resistor_SMD:R_0603_1608Metric_Pad0.98x0.95mm_HandSolder
- R20: renamed from R7; footprint (none) -> Resistor_SMD:R_0603_1608Metric_Pad0.98x0.95mm_HandSolder
- R21: renamed from R15; footprint (none) -> Resistor_SMD:R_0603_1608Metric_Pad0.98x0.95mm_HandSolder
- R22: renamed from R16; footprint (none) -> Resistor_SMD:R_0603_1608Metric_Pad0.98x0.95mm_HandSolder
- R3: renamed from R6; footprint (none) -> Resistor_SMD:R_0603_1608Metric_Pad0.98x0.95mm_HandSolder
- R4: renamed from R1; footprint (none) -> Resistor_SMD:R_0603_1608Metric_Pad0.98x0.95mm_HandSolder
- R5: renamed from R2; footprint (none) -> Resistor_SMD:R_0603_1608Metric_Pad0.98x0.95mm_HandSolder
- R6: renamed from R4; footprint (none) -> Resistor_SMD:R_0603_1608Metric_Pad0.98x0.95mm_HandSolder
- R7: renamed from R5; footprint (none) -> Resistor_SMD:R_0603_1608Metric_Pad0.98x0.95mm_HandSolder
- R8: renamed from R11; footprint (none) -> Resistor_SMD:R_0603_1608Metric_Pad0.98x0.95mm_HandSolder
- R9: renamed from R18; footprint (none) -> Resistor_SMD:R_0603_1608Metric_Pad0.98x0.95mm_HandSolder
- SW1: renamed from SW2; footprint (none) -> Button_Switch_THT:SW_PUSH_6mm
- SW2: renamed from SW1; footprint (none) -> Button_Switch_THT:SW_PUSH_6mm
- renumbered U2 to U1, U8 to U10, U9 to U2, U4 to U3, U5 to U4, U1 to U5, U10 to U6, U3 to U7, U7 to U8, U6 to U9
Connections:
- net GND: now also C14.2, C15.2
- net RXD: no longer names the net of U5.11 (IO20/RXD)
- net TXD: no longer names the net of U5.12 (IO21/TXD)
- no-connect marks 0 -> 3
Other:
- moved on the sheet: C11, C12, C13, J3, R14, R15, R16, R17, R18, R19, R20, U6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

Commit message: Layout attempt two. Routing started
Parts:
- removed H1, H2, H3: MountingHole, MountingHole:MountingHole_2.2mm_M2, symbol Mechanical:MountingHole
- added C22, C23: 1uF, Capacitor_SMD:C_0603_1608Metric_Pad1.08x0.95mm_HandSolder, symbol Device:C
- added H1, H2, H3: MountingHole_Pad, MountingHole:MountingHole_2.2mm_M2_Pad_Via, symbol Mechanical:MountingHole_Pad
- added TP1, TP10, TP11, TP12, TP13, TP14, TP15, TP16, TP17, TP18, TP19, TP2, TP3, TP4, TP5, TP6, TP7, TP8, TP9: TestPoint, TestPoint:TestPoint_THTPad_D1.5mm_Drill0.7mm, symbol Connector:TestPoint
Connections:
- net +1V8: now also C23.1, TP3.1
- net +3V3: now also C22.1, TP2.1
- net +BATT: now also TP1.1
- net +USB_VBUS: now also TP16.1
- net +USB_VBUSF: now also TP17.1
- net BMP_INT: now also TP13.1
- net BOOT_SEL_GPIO9: now also TP18.1
- net CURR_SENSE: now also TP11.1
- net ESP32_EN: now also TP19.1
- net GND: now also C22.2, C23.2, H1.1, H2.1, H3.1
- net I2C_SCL: now also TP9.1
- net I2C_SCL_1V8: now also TP7.1
- net I2C_SDA: now also TP8.1
- net I2C_SDA_1V8: now also TP6.1
- net LSM_INT1: now also TP14.1
- net LSM_INT2: now also TP15.1
- net MAX_INT: now also TP12.1
- net VBATT_SENSE: now also TP10.1
- net at C6.1, D3.1 (K), Q2.2 (S)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: now also TP5.1
- net at C5.1, D2.1 (K), Q1.2 (S)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: now also TP4.1

Commit message: Responding to comments
Parts:
- removed R17: 5k1, Resistor_SMD:R_0603_1608Metric_Pad0.98x0.95mm_HandSolder, symbol Device:R
- removed U7: INA180A1, Package_TO_SOT_SMD:SOT-23-5, symbol Amplifier_Current:INA180A1
- added C24: 0u1, Capacitor_SMD:C_0603_1608Metric_Pad1.08x0.95mm_HandSolder, symbol Device:C
- added R23: 5k1, Resistor_SMD:R_0603_1608Metric_Pad0.98x0.95mm_HandSolder, symbol Device:R
- added U7: INA180A2, Package_TO_SOT_SMD:SOT-23-5, symbol Amplifier_Current:INA180A2
- C1, C2: value 10uF -> 4u7
- C14: value 10uF -> 100n
- C15: value 0u1F -> 100n
- C16: value 0u1F -> 4u7
- C17, C18: value 0u1F -> 0u1
- C19: value 1uF -> 10u
- C5, C6: value 10uF -> 1uF
- R13, R15, R2: value 5k1 -> 1k5
- R16: value 5k1 -> 10k
Connections:
- net +1V8: no longer R16.1
- net +3V3: now also C24.1, R23.1, U7.5 (V+)
- net +BATT: now also U7.4 (-)
- net CURR_SENSE: now also R16.2; no longer TP11.1
- net GND: now also C24.2, U7.2 (GND)
- net I2C_SCL: no longer R15.2
- net I2C_SCL_1V8: no longer R16.2
- net I2C_SDA: no longer R14.2
- net MAX_INT: now also R14.2
- net USB_D+: now also R15.2
- net at J3.1 (Pin_1), R20.2: now also U7.3 (+)
- net at U5.16 (IO2): now also R23.2
- new net: R16.1, TP11.1, U7.1
- no-connect marks 3 -> 2
Other:
- note added: "Note: MAX_INT pin is OD"
- company: UWaterloo -> (none)
- moved on the sheet: J3, R20, TP16, TP6, TP7, TP8, TP9
